Commit message: Updated urdf

File: open_manipulator_description/urdf/open_manipulator.urdf.xacro (robot description, xacro)
@@ -121,22 +121,22 @@
   <joint name="joint4" type="revolute">
     <parent link="link4"/>
-    <child link="link5"/>
+    <child link="link4a"/>
     <origin xyz="0.124 0.0 0.0" rpy="0 0 0"/>
     <axis xyz="0 1 0"/>
     <limit velocity="4.8" effort="1" lower="${-pi*0.57}" upper="${pi*0.65}" />
   </joint>
-  <!--  Link 5 -->
-  <link name="link5">
-    <visual>
-      <origin xyz="0 0 0" rpy="0 0 0"/>
-      <geometry>
-        <mesh filename="package://open_manipulator_description/meshes/chain_link5.stl" scale="0.001 0.001 0.001"/>
-      </geometry>
-      <material name="grey"/>
-    </visual>
-    <collision>
-      <origin xyz="0 0 0" rpy="0 0 0"/>
-      <geometry>
-        <mesh filename="package://open_manipulator_description/meshes/chain_link5.stl" scale="0.001 0.001 0.001"/>
+  <!-- Link 4a-->
+  <link name="link4a">
+    <visual>
+      <origin xyz="0 0 0" rpy="0 0 -1.57"/>
+      <geometry>
+        <mesh filename="package://open_manipulator_description/meshes/chain_link4a.stl" scale="0.001 0.001 0.001"/>
+      </geometry>
+      <material name="grey"/>
+    </visual>
+    <collision>
+      <origin xyz="0 0 0" rpy="0 0 -1.57"/>
+      <geometry>
+        <mesh filename="package://open_manipulator_description/meshes/chain_link4a.stl" scale="0.001 0.001 0.001"/>
       </geometry>
     </collision>
@@ -149,4 +149,35 @@
     </inertial>
   </link>
+  <joint name="joint4a" type="revolute">
+    <parent link="link4a"/>
+    <child link="link5"/>
+    <origin xyz="0.124 0.0 0.0" rpy="0 0 0"/>
+    <axis xyz="1 0 0"/>
+    <limit velocity="4.8" effort="1" lower="${-pi*0.57}" upper="${pi*0.65}" />
+  </joint>
+  <!--  Link 5 -->
+  <!-- pose xyz=0.01 0 0 rpy=1.57 0 0 -->
+  <link name="link5">
+    <visual>
+      <origin xyz="-0.272 0 -0.2045" rpy="1.57 0 0"/>
+      <geometry>
+        <mesh filename="package://open_manipulator_description/meshes/chain_link5a.stl" scale="0.001 0.001 0.001"/>
+      </geometry>
+      <material name="grey"/>
+    </visual>
+    <collision>
+      <origin xyz="-0.272 0 -0.2045" rpy="1.57 0 0"/>
+      <geometry>
+        <mesh filename="package://open_manipulator_description/meshes/chain_link5a.stl" scale="0.001 0.001 0.001"/>
+      </geometry>
+    </collision>
+    <inertial>
+      <origin xyz="4.4206755e-02 3.6839985e-07 8.9142216e-03" />
+      <mass value="1.4327573e-01" />
+      <inertia ixx="8.0870749e-05" ixy="0.0" ixz="-1.0157896e-06"
+               iyy="7.5980465e-05" iyz="0.0"
+               izz="9.3127351e-05" />
+    </inertial>
+  </link>
   <!--  Gripper joint -->
   <joint name="gripper" type="prismatic">
@@ -158,7 +189,8 @@
   </joint>
   <!--  Gripper link -->
+  <!-- pose xyz = 0.281700 0.021 0.21 -->
   <link name="gripper_link">
     <visual>
-      <origin xyz="0.0 0.0 0" rpy="0 0 0"/>
+      <origin xyz="-0.0837 0.0 0.0055" rpy="0 0 0"/>
       <geometry>
         <mesh filename="package://open_manipulator_description/meshes/chain_link_grip_l.stl" scale="0.001 0.001 0.001"/>
@@ -167,5 +199,5 @@
     </visual>
     <collision>
-      <origin xyz="0.0 0.0 0" rpy="0 0 0"/>
+      <origin xyz="-0.0837 0.0 0.0055" rpy="0 0 0"/>
       <geometry>
         <mesh filename="package://open_manipulator_description/meshes/chain_link_grip_l.stl" scale="0.001 0.001 0.001"/>
@@ -184,5 +216,5 @@
     <parent link="link5"/>
     <child link="gripper_link_sub"/>
-    <origin xyz="0.0817 -0.021 0" rpy="0 0 0"/>
+    <origin xyz="0.1217 -0.021 0.0055" rpy="0 0 0"/>
     <axis xyz="0 -1 0"/>
     <limit velocity="4.8" effort="1" lower="-0.010" upper="0.019" />
@@ -192,5 +224,5 @@
   <link name="gripper_link_sub">
     <visual>
-      <origin xyz="0.0 -0.0 0" rpy="0 0 0"/>
+      <origin xyz="-0.0837 -0.0 0" rpy="0 0 0"/>
       <geometry>
         <mesh filename="package://open_manipulator_description/meshes/chain_link_grip_r.stl" scale="0.001 0.001 0.001"/>
@@ -199,5 +231,5 @@
     </visual>
     <collision>
-      <origin xyz="0.0 -0.0 0" rpy="0 0 0"/>
+      <origin xyz="-0.0837 -0.0 0" rpy="0 0 0"/>
       <geometry>
         <mesh filename="package://open_manipulator_description/meshes/chain_link_grip_r.stl" scale="0.001 0.001 0.001"/>
@@ -213,11 +245,11 @@
   </link>
   <!-- end effector joint -->
-  <joint name="end_effector_joint" type="fixed">
+  <!-- <joint name="end_effector_joint" type="fixed">
     <origin xyz="0.126 0.0 0.0" rpy="0 0 0"/>
     <parent link="link5"/>
     <child link="end_effector_link"/>
-  </joint>
+  </joint> -->
   <!-- end effector link -->
-  <link name="end_effector_link">
+  <!-- <link name="end_effector_link">
     <visual>
       <origin xyz="0 0 0" rpy="0 0 0"/>
@@ -234,5 +266,5 @@
                izz="1.0e-03" />
     </inertial>
-  </link>
+  </link> -->
   <!-- Realsense Camera Joint Position -->
 <!--   <joint name="camera_joint" type="fixed">
